Commit message: fully functioning autonomous navigation simulation.

File: leo_description/urdf/leo.urdf.xacro (robot description, xacro)
@@ -6,4 +6,5 @@
   <xacro:arg name="default_antenna" default="true"/>
   <xacro:arg name="rockers_fixed" default="true"/>
+  <xacro:property name="link_prefix"      value="" />
   <xacro:if value="false">
     <link name="world"/>
@@ -93,4 +94,7 @@
   </link>
   <link name="base_footprint"/>
+  <link name="imu_link">
+  <!-- Frame to attach an IMU to -->
+  </link>
   <xacro:rocker_link name="L"/>
   <xacro:rocker_link name="R"/>
@@ -126,5 +130,5 @@
   <link name="rplidar_link">
     <visual>
-      <origin xyz="0 0 0.003"/>
+      <origin xyz="0 0 0.009"/>
       <geometry>
         <box size="0.079 0.086 0.006"/>
@@ -157,5 +161,5 @@
   </link>
   <joint name="rplidar_joint" type="fixed">
-    <origin xyz="0.0775 0 0"/>
+    <origin xyz="0.0775 0 0.05"/>
     <parent link="base_link"/>
     <child link="rplidar_link"/>
@@ -169,5 +173,10 @@
     <xacro:property name="rockers_joint_type" value="revolute"/>
   </xacro:unless>
-  <joint name="rocker_L_joint" type="revolute"> <!-- ${rockers_joint_type} -->
+  <joint name="imu_joint" type="fixed">
+    <parent link="base_link"/>
+    <child link="imu_link"/>
+    <origin xyz="0 0 0" rpy="0 0 0"/>
+  </joint>
+  <joint name="rocker_L_joint" type="fixed"> <!-- ${rockers_joint_type} -->
     <origin xyz="0.00263 0.14167 -0.04731" rpy="0 0 ${3.141592653589793}"/>
     <parent link="base_link"/>
@@ -177,5 +186,5 @@
     <dynamics friction="1.0" damping="0.1"/>
   </joint>
-  <joint name="rocker_R_joint" type="revolute">
+  <joint name="rocker_R_joint" type="fixed">
     <origin xyz="0.00263 -0.14167 -0.04731" rpy="0 0 0"/>
     <parent link="base_link"/>
@@ -241,5 +250,5 @@
   </joint>
   <joint name="laser_joint" type="fixed">
-    <origin xyz="0 0 0.0368" rpy="0 0 ${pi}"/>
+    <origin xyz="0 0 0.0568" rpy="0 0 ${pi}"/>
     <parent link="rplidar_link"/>
     <child link="laser_frame"/>
@@ -302,52 +311,191 @@
     </transmission>
   </xacro:unless>
-   <!-- rocker differential -->
-    <gazebo>
-      <plugin name="leo_gz::DifferentialSystem" filename="libleo_gz_differential_plugin.so">
-        <jointA>rocker_L_joint</jointA>
-        <jointB>rocker_R_joint</jointB>
-        <forceConstant>100.0</forceConstant>
-      </plugin>
-    </gazebo>
-    <gazebo>
+     <!-- GAZEBO PLUGINS -->
+  <!-- Differential Drive - https://gazebosim.org/api/gazebo/4.5/classignition_1_1gazebo_1_1systems_1_1DiffDrive.html -->
+  <gazebo>
+    <plugin filename="ignition-gazebo-diff-drive-system" name="ignition::gazebo::systems::DiffDrive">
+      <!-- Wheel Joints -->
+      <left_joint>wheel_FL_joint</left_joint>
+        <right_joint>wheel_FR_joint</right_joint>
+        <left_joint>wheel_RL_joint</left_joint>
+        <right_joint>wheel_RR_joint</right_joint>
+      <!-- Kinematics -->
+      <wheel_separation>0.358</wheel_separation>
+        <wheel_radius>0.0625</wheel_radius>
+      <odom_publish_frequency>50</odom_publish_frequency>
+      <!-- TF Frames -->
+      <frame_id>/odom</frame_id>
+      <child_frame_id>base_footprint</child_frame_id>
+      <!-- topics -->
+      <!-- <topic>/model/gz_example_robot/cmd_vel</topic> THIS IS DEFAULT -->
+      <!-- <odom_topic>/model/gz_example_robot/odometry</odom_topic> THIS IS DEFAULT-->
+      <!-- <tf_topic>/model/gz_example_robot/tf</tf_topic> THIS IS DEFAULT -->
+      <!-- <tf_topic></tf_topic> Leave blank if you plan to use a filter + imu (e.g. EKF) -->
+    </plugin>
+  </gazebo>
+     <gazebo>
       <plugin
         filename="ignition-gazebo-joint-state-publisher-system"
         name="ignition::gazebo::systems::JointStatePublisher">
-        <topic>joint_states</topic>
+        <topic>/joint_states</topic>
+        <update_rate>50</update_rate>
+        <joint_name>wheel_FL_joint</joint_name>
+        <joint_name>wheel_FR_joint</joint_name>
+        <joint_name>wheel_RL_joint</joint_name>
+        <joint_name>wheel_RR_joint</joint_name>
       </plugin>
     </gazebo>
-    <gazebo reference="imu_frame">
-      <sensor type="imu" name="leo_imu_sensor">
-        <update_rate>100</update_rate>
-        <visualize>true</visualize>
-        <topic>imu/data_raw</topic>
-        <always_on>1</always_on>
-        <ignition_frame_id>imu_frame</ignition_frame_id>
-      </sensor>
-    </gazebo>
-    <gazebo>
-      <plugin
-        filename="libignition-gazebo-diff-drive-system.so"
-        name="ignition::gazebo::systems::DiffDrive">
-        <left_joint>wheel_FL_joint</left_joint>
-        <right_joint>wheel_FR_joint</right_joint>
-        <left_joint>wheel_RL_joint</left_joint>
-        <right_joint>wheel_RR_joint</right_joint>
-        <wheel_separation>0.358</wheel_separation>
-        <wheel_radius>0.0625</wheel_radius>
-        <frame_id>odom</frame_id>
-        <child_frame_id>base_footprint</child_frame_id>
-        <odom_publish_frequency>20</odom_publish_frequency>
-        <topic>cmd_vel</topic>
-        <odom_topic>odom</odom_topic>
-        <tf_topic>tf</tf_topic>
-        <max_linear_acceleration>2.5</max_linear_acceleration>
-        <max_angular_acceleration>3</max_angular_acceleration>
-        <min_linear_acceleration>-2.5</min_linear_acceleration>
-        <min_angular_acceleration>-3</min_angular_acceleration>
-      </plugin>
-    </gazebo>
-  <!--lidar-->
-  <gazebo reference="rplidar_link">
+   <!-- base ODE properties -->
+    <gazebo reference="base_footprint">
+      <collision>
+        <surface>
+          <friction>
+            <ode>
+              <mu>0.3</mu>
+              <mu2>0.3</mu2>
+            </ode>
+            <bullet>
+              <friction>0.3</friction>
+              <friction2>0.3</friction2>
+              <rolling_friction>0.1</rolling_friction>
+            </bullet>
+          </friction>
+        </surface>
+      </collision>
+    </gazebo>
+    <gazebo reference="base_link">
+      <collision>
+        <surface>
+          <friction>
+            <ode>
+              <mu>0.3</mu>
+              <mu2>0.3</mu2>
+            </ode>
+            <bullet>
+              <friction>0.3</friction>
+              <friction2>0.3</friction2>
+              <rolling_friction>0.1</rolling_friction>
+            </bullet>
+          </friction>
+        </surface>
+      </collision>
+    </gazebo>
+    <!-- rocker ODE properties -->
+    <gazebo reference="rocker_L_link">
+      <collision>
+        <surface>
+          <friction>
+            <ode>
+              <mu>0.3</mu>
+              <mu2>0.3</mu2>
+            </ode>
+            <bullet>
+              <friction>0.3</friction>
+              <friction2>0.3</friction2>
+              <rolling_friction>0.1</rolling_friction>
+            </bullet>
+          </friction>
+        </surface>
+      </collision>
+    </gazebo>
+    <gazebo reference="rocker_R_link">
+      <collision>
+        <surface>
+          <friction>
+            <ode>
+              <mu>0.3</mu>
+              <mu2>0.3</mu2>
+            </ode>
+            <bullet>
+              <friction>0.3</friction>
+              <friction2>0.3</friction2>
+              <rolling_friction>0.1</rolling_friction>
+            </bullet>
+          </friction>
+        </surface>
+      </collision>
+    </gazebo>
+    <!-- wheel ODE properties -->
+    <gazebo reference="wheel_FL_link">
+      <collision>
+        <surface>
+          <friction>
+            <ode>
+              <mu>1</mu>
+              <mu2>1</mu2>
+              <slip1>0.035</slip1>
+              <slip2>0</slip2>
+              <fdir1>0 0 1</fdir1>
+            </ode>
+            <bullet>
+              <friction>1</friction>
+              <friction2>1</friction2>
+              <rolling_friction>0.1</rolling_friction>
+            </bullet>
+          </friction>
+        </surface>
+      </collision>
+    </gazebo>
+    <gazebo reference="wheel_FR_link">
+      <collision>
+        <surface>
+          <friction>
+            <ode>
+              <mu>1</mu>
+              <mu2>1</mu2>
+              <slip1>0.035</slip1>
+              <slip2>0</slip2>
+              <fdir1>0 0 1</fdir1>
+            </ode>
+            <bullet>
+              <friction>1</friction>
+              <friction2>1</friction2>
+              <rolling_friction>0.1</rolling_friction>
+            </bullet>
+          </friction>
+        </surface>
+      </collision>
+    </gazebo>
+    <gazebo reference="wheel_RL_link">
+      <collision>
+        <surface>
+          <friction>
+            <ode>
+              <mu>1</mu>
+              <mu2>1</mu2>
+              <slip1>0.035</slip1>
+              <slip2>0</slip2>
+              <fdir1>0 0 1</fdir1>
+            </ode>
+            <bullet>
+              <friction>1</friction>
+              <friction2>1</friction2>
+              <rolling_friction>0.1</rolling_friction>
+            </bullet>
+          </friction>
+        </surface>
+      </collision>
+    </gazebo>
+    <gazebo reference="wheel_RR_link">
+      <collision>
+        <surface>
+          <friction>
+            <ode>
+              <mu>1</mu>
+              <mu2>1</mu2>
+              <slip1>0.035</slip1>
+              <slip2>0</slip2>
+              <fdir1>0 0 1</fdir1>
+            </ode>
+            <bullet>
+              <friction>1</friction>
+              <friction2>1</friction2>
+              <rolling_friction>0.1</rolling_friction>
+            </bullet>
+          </friction>
+        </surface>
+      </collision>
+    </gazebo>
+    <gazebo reference="rplidar_link">
     <sensor type="gpu_lidar" name="generic_lidar_sensor">
       <topic>/model/leo/scan</topic>
@@ -384,3 +532,70 @@
     </plugin>
   </gazebo>
+  <gazebo reference="imu_link">
+    <sensor name="imu_sensor" type="imu">
+      <topic>/model/leo/imu</topic>
+      <frame_id>imu_link</frame_id>
+      <ignition_frame_id>imu_link</ignition_frame_id>
+      <plugin filename="libignition-gazebo-imu-system.so" name="ignition::gazebo::systems::Imu">
+        <initial_orientation_as_reference>false</initial_orientation_as_reference>
+      </plugin>
+      <always_on>true</always_on>
+      <update_rate>100</update_rate>
+      <visualize>true</visualize>
+     <imu>
+     	<angular_velocity>
+     	  <x>
+     	    <noise type="gaussian">
+              <mean>0.0</mean>
+              <stddev>2e-4</stddev>
+              <bias_mean>0.0000075</bias_mean>
+              <bias_stddev>0.0000008</bias_stddev>
+            </noise>
+          </x>
+          <y>
+            <noise type="gaussian">
+              <mean>0.0</mean>
+              <stddev>2e-4</stddev>
+              <bias_mean>0.0000075</bias_mean>
+              <bias_stddev>0.0000008</bias_stddev>
+            </noise>
+          </y>
+          <z>
+            <noise type="gaussian">
+              <mean>0.0</mean>
+              <stddev>2e-4</stddev>
+              <bias_mean>0.0000075</bias_mean>
+              <bias_stddev>0.0000008</bias_stddev>
+            </noise>
+          </z>
+        </angular_velocity>
+        <linear_acceleration>
+          <x>
+            <noise type="gaussian">
+              <mean>0.0</mean>
+              <stddev>1.7e-2</stddev>
+              <bias_mean>0.1</bias_mean>
+              <bias_stddev>0.001</bias_stddev>
+            </noise>
+          </x>
+          <y>
+            <noise type="gaussian">
+              <mean>0.0</mean>
+              <stddev>1.7e-2</stddev>
+              <bias_mean>0.1</bias_mean>
+              <bias_stddev>0.001</bias_stddev>
+            </noise>
+          </y>
+          <z>
+            <noise type="gaussian">
+              <mean>0.0</mean>
+              <stddev>1.7e-2</stddev>
+              <bias_mean>0.1</bias_mean>
+              <bias_stddev>0.001</bias_stddev>
+            </noise>
+          </z>
+        </linear_acceleration>
+      </imu>
+    </sensor>
+  </gazebo>
 </robot>

File: leo_description/urdf/leo_proper.gazebo.xacro (robot description, xacro)
@@ -2,18 +2,4 @@
 <robot xmlns:xacro="http://ros.org/wiki/xacro">
   <!-- rocker differential -->
-    <gazebo>
-      <plugin name="leo_gz::DifferentialSystem" filename="libleo_gz_differential_plugin.so">
-        <jointA>rocker_L_joint</jointA>
-        <jointB>rocker_R_joint</jointB>
-        <forceConstant>100.0</forceConstant>
-      </plugin>
-    </gazebo>
-    <gazebo>
-      <plugin
-        filename="ignition-gazebo-joint-state-publisher-system"
-        name="ignition::gazebo::systems::JointStatePublisher">
-        <topic>oint_states</topic>
-      </plugin>
-    </gazebo>
     <gazebo reference="imu_frame">
       <sensor type="imu" name="leo_imu_sensor">
@@ -25,4 +11,71 @@
       </sensor>
     </gazebo>
+    <gazebo reference="imu_link">
+    <sensor name="imu_sensor" type="imu">
+      <topic>/imu/data_raw</topic>
+      <frame_id>imu_link</frame_id>
+      <ignition_frame_id>imu_link</ignition_frame_id>
+      <plugin filename="libignition-gazebo-imu-system.so" name="ignition::gazebo::systems::Imu">
+        <initial_orientation_as_reference>false</initial_orientation_as_reference>
+      </plugin>
+      <always_on>true</always_on>
+      <update_rate>100</update_rate>
+      <visualize>true</visualize>
+     <imu>
+     	<angular_velocity>
+     	  <x>
+     	    <noise type="gaussian">
+              <mean>0.0</mean>
+              <stddev>2e-4</stddev>
+              <bias_mean>0.0000075</bias_mean>
+              <bias_stddev>0.0000008</bias_stddev>
+            </noise>
+          </x>
+          <y>
+            <noise type="gaussian">
+              <mean>0.0</mean>
+              <stddev>2e-4</stddev>
+              <bias_mean>0.0000075</bias_mean>
+              <bias_stddev>0.0000008</bias_stddev>
+            </noise>
+          </y>
+          <z>
+            <noise type="gaussian">
+              <mean>0.0</mean>
+              <stddev>2e-4</stddev>
+              <bias_mean>0.0000075</bias_mean>
+              <bias_stddev>0.0000008</bias_stddev>
+            </noise>
+          </z>
+        </angular_velocity>
+        <linear_acceleration>
+          <x>
+            <noise type="gaussian">
+              <mean>0.0</mean>
+              <stddev>1.7e-2</stddev>
+              <bias_mean>0.1</bias_mean>
+              <bias_stddev>0.001</bias_stddev>
+            </noise>
+          </x>
+          <y>
+            <noise type="gaussian">
+              <mean>0.0</mean>
+              <stddev>1.7e-2</stddev>
+              <bias_mean>0.1</bias_mean>
+              <bias_stddev>0.001</bias_stddev>
+            </noise>
+          </y>
+          <z>
+            <noise type="gaussian">
+              <mean>0.0</mean>
+              <stddev>1.7e-2</stddev>
+              <bias_mean>0.1</bias_mean>
+              <bias_stddev>0.001</bias_stddev>
+            </noise>
+          </z>
+        </linear_acceleration>
+      </imu>
+    </sensor>
+  </gazebo>
     <gazebo>
       <plugin
@@ -83,4 +136,56 @@
     </plugin>
   </gazebo>
+    <gazebo>
+      <plugin
+        filename="ignition-gazebo-joint-state-publisher-system"
+        name="ignition::gazebo::systems::JointStatePublisher">
+        <topic>joint_states</topic>
+      </plugin>
+    </gazebo>
+    <gazebo reference="imu_frame">
+      <sensor type="imu" name="leo_imu_sensor">
+        <update_rate>100</update_rate>
+        <visualize>true</visualize>
+        <topic>imu/data_raw</topic>
+        <always_on>1</always_on>
+        <ignition_frame_id>imu_frame</ignition_frame_id>
+      </sensor>
+    </gazebo>
+  <!--lidar-->
+  <gazebo reference="rplidar_link">
+    <sensor type="gpu_lidar" name="generic_lidar_sensor">
+      <topic>/model/leo/scan</topic>
+      <frame_id>rplidar_link</frame_id>
+      <ignition_frame_id>rplidar_link</ignition_frame_id>
+      <update_rate>10.0</update_rate>
+      <ray>
+        <scan>
+          <horizontal>
+            <samples>512</samples>
+            <resolution>1</resolution>
+            <min_angle>-${pi*2}</min_angle>
+            <max_angle>${pi*2}</max_angle>
+          </horizontal>
+        </scan>
+        <range>
+          <min>0.10</min>
+          <max>10.0</max>
+          <resolution>0.03</resolution>
+        </range>
+        <noise>
+          <type>gaussian</type>
+          <mean>0.0</mean>
+          <stddev>0.001</stddev>
+        </noise>
+      </ray>
+      <always_on>1</always_on>
+      <visualize>false</visualize>
+    </sensor>
+  </gazebo>
+  <gazebo>
+    <plugin filename="libignition-gazebo-sensors-system.so" name="ignition::gazebo::systems::Sensors">
+      <render_engine>ogre2</render_engine>
+    </plugin>
+  </gazebo>
   <gazebo reference="imu_link">
     <sensor name="imu_sensor" type="imu">

Commit message: square map added and lidar on the belly, with scan malware

File: leo_description/urdf/leo.urdf.xacro (robot description, xacro)
@@ -161,9 +161,28 @@
   </link>
   <joint name="rplidar_joint" type="fixed">
-    <origin xyz="0.0775 0 0.05"/>
+    <origin xyz="0.0 0 -0.1" rpy = "${pi} 0 0"/>
     <parent link="base_link"/>
     <child link="rplidar_link"/>
   </joint>
   <link name="laser_frame"/>
+  <link name="depth_camera_link">
+        <visual>
+            <geometry>
+                <box size="0.02 0.08 0.016"/>
+            </geometry>
+            <material name="green">
+                <color rgba="0 1 0 1"/>
+            </material>
+        </visual>
+        <collision>
+            <geometry>
+                <box size="0.02 0.08 0.016"/>
+            </geometry>
+        </collision>
+        <inertial>
+          <mass value="4.2"/>
+          <inertia ixx="0.00004533" ixy="0.0" ixz="0.0" iyy="0.000004373" iyz="0.0" izz="0.00004437"/>
+        </inertial>
+    </link>
   <!-- JOINTS -->
   <xacro:if value="true">
@@ -254,4 +273,9 @@
     <child link="laser_frame"/>
   </joint>
+  <joint name="chassis_depth_camera_joint" type="fixed">
+        <parent link="base_link"/>
+        <child link="depth_camera_link"/>
+        <origin xyz="0.0971 0 0.0227" rpy="0 0 0"/>
+    </joint>
   <!-- TRANSMISSIONS -->
   <transmission name="wheel_FL_trans">
@@ -499,5 +523,5 @@
     <gazebo reference="rplidar_link">
     <sensor type="gpu_lidar" name="generic_lidar_sensor">
-      <topic>/model/leo/scan</topic>
+      <topic>/model/leo/scan_e</topic>
       <frame_id>rplidar_link</frame_id>
       <ignition_frame_id>rplidar_link</ignition_frame_id>
@@ -508,10 +532,10 @@
             <samples>512</samples>
             <resolution>1</resolution>
-            <min_angle>-${pi*2}</min_angle>
+            <min_angle>${-pi*2}</min_angle>
             <max_angle>${pi*2}</max_angle>
           </horizontal>
         </scan>
         <range>
-          <min>0.10</min>
+          <min>0.001</min>
           <max>10.0</max>
           <resolution>0.03</resolution>
@@ -532,4 +556,27 @@
     </plugin>
   </gazebo>
+  <gazebo reference="depth_camera_link">
+  <sensor name="william_harvey_depth_camera" type="depth_camera">
+  <topic>/model/leo/depth_camera</topic>
+  <frame_id>depth_camera_link</frame_id>
+  <ignition_frame_id>depth_camera_link</ignition_frame_id>
+    <update_rate>10</update_rate>
+    <camera name="simple_camera">
+              <horizontal_fov>1.51855</horizontal_fov>
+              <vertical_fov>1.01229</vertical_fov>
+              <image>
+                  <width>1280</width>
+                  <height>720</height>
+                  <format>R8G8B8</format>
+              </image>
+              <clip>
+              <near>0.1</near>
+              <far>2.0</far>
+              </clip>
+          </camera>
+          <always_on>1</always_on>
+          <visualize>true</visualize>
+      </sensor>
+    </gazebo>
   <gazebo reference="imu_link">
     <sensor name="imu_sensor" type="imu">
